File: pcb/same51-dev.sch (EAGLE design)
At the start: 41 parts, among them U1 ATSAMD51J, U2 W25Q40BVSS, U3 MCP1631TDFN8, U4 MCP2562-MF, X1 32.768kHz

Commit message: finished sch, started pcb
Parts:
- added C20, C22: 100n, Passive Components > Capacitors > Multilayer Ceramic Capacitors MLCC:MLCC0603
- added C21: 4n4, Passive Components > Capacitors > Multilayer Ceramic Capacitors MLCC:MLCC0603
- added D3: SP0503BAHT, Circuit Protection > ESD Suppressors \ TVS Diodes:SP0503BAHT
- added J1: 4, Connectors > Header:4
- added J10, J4, J5, J7, J8: 8, Connectors > Header:8
- added J2: USB-C, Connectors > USB:USB-C
- added J3: 6, Connectors > Header:6
- added J6: 3, Connectors > Header:3
- added J9: 5, Connectors > Header:5
- added R11, R12: 11k5, Passive Components > Resistors > Chip Resistors:RESISTOR0603
- added R13: 1M, Passive Components > Resistors > Chip Resistors:RESISTOR0603
- added SW1: (no value), Eletromechanical > Switches > Tactile Switches:PUSH_BUTTON3X4X2
- added SW2: MSK-13C01, Eletromechanical > Switches > Toggle Switches:MSK-13C01
Connections:
- removed net DM: U1.PA.PA24/I8/SERCOM3+5.2/D-
- removed net DP: U1.PA.PA25/19/SERCOM3+5.3/D+
- removed net N$6: C17.P$1, C18.P$1, F1.1, U3.EN, U3.VIN
- removed net PA22: U1.PA.PA22/I2C/16/SERCOM3.0+5.1/I2SDI
- removed net PA23: U1.PA.PA23/I2C/I7/SERCOM3.1+5.0/SOF/I2SFS1
- new net CAN_RX: J5-8.S, U1.PA.PA23/I2C/I7/SERCOM3.1+5.0/SOF/I2SFS1, U4.RXD
- new net CAN_TX: J5-7.S, U1.PA.PA22/I2C/16/SERCOM3.0+5.1/I2SDI, U4.TXD
- new net N$11: J1-2.S, U4.CANH
- new net N$13: C21.P$1, D3.1, J2.SHIELD, R13.P$2
- new net N$15: J2.CC2@B5, R11.P$2
- new net N$16: J2.CC1@A5, R12.P$2
- new net N$9: J1-3.S, U4.CANL
- new net USB_DM: D3.4, J2.DN@A7,B7, J6-1.S, U1.PA.PA24/I8/SERCOM3+5.2/D-
- new net USB_DP: D3.3, J2.DP@A6,B6, J6-2.S, U1.PA.PA25/19/SERCOM3+5.3/D+
- new net VCC: C22.P$1, J1-1.S, SW2.2, U4.VDD
- new net VDD: C17.P$1, C18.P$1, F1.1, J10-4.S, J10-5.S, U3.EN, U3.VIN
- new net VSUP: SW2.4
- new net VUSB: D3.2, J2.VBUS@A4,A9,B9,B4, SW2.1
- net !RESET: now also SW1.4
- net 3.3V: now also C20.P$1, J10-1.S, J10-2.S, J10-3.S, U4.VIO
- net GND: now also C20.P$2, C21.P$2, C22.P$2, J1-4.S, J10-6.S, J10-7.S, J10-8.S, J2.GND@A1,A12,B12,B1, R11.P$1, R12.P$1, R13.P$1, SW1.1, SW1.2, U4.STDBY, U4.VSS
- net LED: now also J6-3.S
- net PA02: now also J3-1.S
- net PA03: now also J3-2.S
- net PA04: now also J3-3.S
- net PA05: now also J3-4.S
- net PA06: now also J3-5.S
- net PA07: now also J3-6.S
- net PA14: now also J4-7.S
- net PA15: now also J4-8.S
- net PA16: now also J5-1.S
- net PA17: now also J5-2.S
- net PA18: now also J5-3.S
- net PA19: now also J5-4.S
- net PA20: now also J5-5.S
- net PA21: now also J5-6.S
- net PB00: now also J7-1.S
- net PB01: now also J7-2.S
- net PB02: now also J7-3.S
- net PB03: now also J7-4.S
- net PB04: now also J7-5.S
- net PB05: now also J7-6.S
- net PB06: now also J7-7.S
- net PB07: now also J7-8.S
- net PB08: now also J8-1.S
- net PB09: now also J8-2.S
- net PB12: now also J8-5.S
- net PB13: now also J8-6.S
- net PB14: now also J8-7.S
- net PB15: now also J8-8.S
- net PB16: now also J9-1.S
- net PB17: now also J9-2.S
- net PB22: now also J9-3.S
- net PB23: now also J9-4.S
- net PB31: now also J9-5.S
- net QSPI_CS: now also J8-4.S
- net QSPI_IO0: now also J4-1.S
- net QSPI_IO1: now also J4-2.S
- net QSPI_IO2: now also J4-3.S
- net QSPI_IO3: now also J4-4.S
- net QSPI_SCK: now also J8-3.S
- net SCL: now also J4-6.S
- net SDA: now also J4-5.S
- net VIN: now also SW2.3
Other:
- note added: "U4-3"
- note added: "U4-5"
- moved on the sheet: C11, C12, D1, D2, R5, R6, R7, R8, U4, X1

Commit message: power routing
Parts:
- added J11: 2, Connectors > Header:2
Connections:
- net GND: now also J11-2.S
- net VSUP: now also J11-1.S
Changed lines of the file:
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@@
 <part name="SUPPLY23" library="Utility &gt; Power Symbols" deviceset="VDD" device=""/>
 <part name="SUPPLY29" library="Utility &gt; Power Symbols" deviceset="VDD" device=""/>
+<part name="J11" library="Connectors &gt; Header" deviceset="2" device=""/>
+<part name="SUPPLY30" library="Utility &gt; Power Symbols" deviceset="VSUP" device=""/>
+<part name="GND34" library="Utility &gt; Power Symbols" deviceset="GND" device=""/>
 </parts>
 <sheets>
@@
 <attribute name="VALUE" x="274.32" y="162.814" size="1.778" layer="96" align="bottom-center"/>
 </instance>
+<instance part="J11" gate="-1" x="218.44" y="165.1" smashed="yes">
+<attribute name="NAME" x="220.98" y="164.338" size="1.524" layer="95"/>
+</instance>
+<instance part="J11" gate="-2" x="218.44" y="162.56" smashed="yes">
+<attribute name="NAME" x="220.98" y="161.798" size="1.524" layer="95"/>
+</instance>
+<instance part="SUPPLY30" gate="G$1" x="213.36" y="165.1" smashed="yes">
+<attribute name="VALUE" x="213.36" y="167.894" size="1.778" layer="96" align="bottom-center"/>
+</instance>
+<instance part="GND34" gate="1" x="213.36" y="160.02" smashed="yes">
+<attribute name="VALUE" x="213.36" y="159.766" size="1.778" layer="96" align="top-center"/>
+</instance>
 </instances>
 <busses>
@@
 <pinref part="J10" gate="-8" pin="S"/>
 </segment>
+<segment>
+<pinref part="GND34" gate="1" pin="GND"/>
+<pinref part="J11" gate="-2" pin="S"/>
+<wire x1="213.36" y1="162.56" x2="215.9" y2="162.56" width="0.1524" layer="91"/>
+</segment>
 </net>
 <net name="3.3V" class="0">
@@
 <pinref part="SUPPLY27" gate="G$1" pin="VSUP"/>
 </segment>
-</net>
+<segment>
+<pinref part="J11" gate="-1" pin="S"/>
+<wire x1="215.9" y1="165.1" x2="213.36" y2="165.1" width="0.1524" layer="91"/>
+<pinref part="SUPPLY30" gate="G$1" pin="VSUP"/>
+</segment>
+</net>
