File: pcb/same51-dev.brd (EAGLE design)
At the start: 83.5 x 68.2 mm, 60 parts, among them J1 4, J10 8, J2 USB-C, J3 6, J4 8, J5 8, J6 3, J7 8, J8 8, J9 5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

Commit message: power routing
Parts:
- added J11: 2, Connectors > Header:2X1_2.54
- moved C7 1.96 mm to (33.6, 16.3), turned to 270 degrees
- moved C6 1.23 mm to (40.6, 16.4), turned to 270 degrees
- moved C11 0.30 mm to (46.7, 35.6)
- moved C12 0.30 mm to (39.7, 35.6)
- turned SW1 to 180 degrees
Connections:
- net GND: now also J11.2
- net VSUP: now also J11.1
Routing:
- net 3.3V: track 0.00 -> 224.6 mm, vias 0 -> 2
- net VDD: track 0.00 -> 63.3 mm, vias 0 -> 2
- net VCC: track 0.00 -> 62.2 mm, vias 0 -> 1
- net USB_DM: track 0.00 -> 60.6 mm, vias 0 -> 3
- net !RESET: track 0.00 -> 56.1 mm, vias 0 -> 2
- net USB_DP: track 0.00 -> 56.0 mm, vias 0 -> 2
- net SWO: track 0.00 -> 49.2 mm, vias 0 -> 2
- net SWDIO: track 0.00 -> 45.0 mm, vias 0 -> 2
- net SWCLK: track 0.00 -> 44.3 mm, vias 0 -> 2
- net VUSB: track 0.00 -> 38.0 mm, vias 0 -> 2
- net CAN_TX: track 0.00 -> 37.7 mm, vias 0 -> 2
- net LED: track 0.00 -> 37.3 mm, vias 0 -> 3
- net CAN_RX: track 0.00 -> 35.8 mm, vias 0 -> 2
- net VIN: track 0.00 -> 15.3 mm, vias 0 -> 2
- net N$16: track 0.00 -> 14.4 mm, vias 0 -> 2
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Other:
- board text added: "VSUP"
- board text removed: "PIN"

Commit message: finished signal routing
Parts:
- moved C7 0.70 mm to (33.6, 15.6)
- moved C8 0.70 mm to (28.5, 26.7)
Routing:
- net PB12: track 0.00 -> 92.1 mm, vias 0 -> 1
- net PB13: track 0.00 -> 89.7 mm, vias 0 -> 1
- net PB14: track 0.00 -> 88.0 mm, vias 0 -> 1
- net PB15: track 0.00 -> 84.5 mm, vias 0 -> 1
- net PB17: track 0.00 -> 83.0 mm, vias 0 -> 1
- net PB16: track 0.00 -> 78.5 mm, vias 0 -> 1
- net QSPI_SCK: track 13.1 -> 87.5 mm, vias 2 -> 3
- net QSPI_CS: track 17.2 -> 90.8 mm
- net PA02: track 0.00 -> 67.6 mm, vias 0 -> 3
- net PA03: track 0.00 -> 63.3 mm, vias 0 -> 2
- net SDA: track 0.00 -> 59.7 mm, vias 0 -> 1
- net SCL: track 0.00 -> 57.5 mm, vias 0 -> 1
- net PB08: track 0.00 -> 57.3 mm, vias 0 -> 3
- net PB22: track 0.00 -> 56.1 mm, vias 0 -> 1
- net PB09: track 0.00 -> 54.1 mm, vias 0 -> 2
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
Commit message: V1.0 Ready for production
Parts:
- added U$1: (no value), Utility > Silkscreen:OSHW-LOGO-L
- added U$2: (no value), Utility > Silkscreen:RAFAEL_SILVA_10MM_ALT
- added U$3: (no value), Utility > Silkscreen:RAFAEL_SILVA_5MM_ALT_3
- added U$4: (no value), Utility > Silkscreen:OSHW-LOGO-M
- moved C6 0.61 mm to (40.6, 15.8)
- flipped J3 to the top
- flipped J10 to the top
Routing:
- net 3.3V: track 224.7 -> 238.4 mm
- net GND: track 0.00 -> 1.68 mm, vias 0 -> 721
- net PB06: track 31.0 -> 30.4 mm
- added copper zone on layer 1, net GND
- added copper zone on layer 16, net GND
Other:
- board text added: "*"
- board text added: "* = special funcion"
- board text added: "15V Max"
- board text added: "5V5 Max"
- board text added: "ATSAME51"
- board text added: "CC"
- board text added: "Designed in Portugal"
- board text added: "IO0"
- board text added: "IO1"
- board text added: "IO2"
- board text added: "IO3"
- board text added: "PA08"
- board text added: "PA09"
- board text added: "PA10"
- board text added: "PA11"
- board text added: "PA12"
- board text added: "PA13"
- board text added: "PA14"
- board text added: "PA15"
- board text added: "PA16"
- board text added: "PA17"
- board text added: "PA18"
- board text added: "PA19"
- board text added: "PA20"
- board text added: "PA21"
- board text added: "PA22"
- board text added: "PA23"
- board text added: "PA24"
- board text added: "PA25"
- board text added: "PA26"
- board text added: "PB00"
- board text added: "PB01"
- board text added: "PB02"
- board text added: "PB03"
- board text added: "PB04"
- board text added: "PB05"
- board text added: "PB06"
- board text added: "PB07"
- board text added: "PB08"
- board text added: "PB09"
- board text added: "PB10"
- board text added: "PB11"
- board text added: "PB12"
- board text added: "PB13"
- board text added: "PB14"
- board text added: "PB15"
- board text added: "PB16"
- board text added: "PB17"
- board text added: "PB22"
- board text added: "PB23"
- board text added: "PB31"
- board text added: "Q CS"
- board text added: "Q SCK"
- board text added: "QSPI"
- board text added: "RX"
- board text added: "SAME51-DevBoard V1.0 #5019"
- board text added: "SCL"
- board text added: "SDA"
- board text added: "TX"
- board text added: "github/gimbas"
